Commit message: Created Multi Robot Simulation System

File: urdf/robot.urdf (robot description, URDF)
Before this commit: robot diff_drive_robot, 7 links, 6 joints
Links:
- removed link base_link
- removed link castor_wheel
- removed link chassis
- removed link imu_link
- removed link laser_frame
- removed link left_wheel
- removed link right_wheel
- added link robot_2_base_footprint; visual sphere radius=0.01
- added link robot_2_base_link, mass 0.5; collision box size=0.3 0.3 0.15; visual box size=0.3 0.3 0.15
- added link robot_2_castor_wheel, mass 0.05; collision sphere radius=0.05; visual sphere radius=0.05
- added link robot_2_imu_link; visual box size=0.02 0.02 0.02
- added link robot_2_laser_frame, mass 0.1; collision cylinder length=0.04 radius=0.05; visual cylinder length=0.04 radius=0.05
- added link robot_2_left_wheel, mass 0.1; collision cylinder length=0.04 radius=0.05; visual cylinder length=0.04 radius=0.05
- added link robot_2_right_wheel, mass 0.1; collision cylinder length=0.04 radius=0.05; visual cylinder length=0.04 radius=0.05
Joints:
- removed joint castor_wheel_joint
- removed joint chassis_joint
- removed joint imu_joint
- removed joint laser_joint
- removed joint left_wheel_joint
- removed joint right_wheel_joint
- added joint robot_2_base_joint: type fixed, parent robot_2_base_footprint, child robot_2_base_link, origin xyz=0 0 0.075 rpy=0 0 0
- added joint robot_2_castor_wheel_joint: type fixed, parent robot_2_base_link, child robot_2_castor_wheel, origin xyz=0.15 0 -0.075
- added joint robot_2_imu_joint: type fixed, parent robot_2_base_footprint, child robot_2_imu_link, origin xyz=0 0 0.075 rpy=0 0 0
- added joint robot_2_laser_joint: type fixed, parent robot_2_base_link, child robot_2_laser_frame, origin xyz=0.15 0 0.075 rpy=0 0 0
- added joint robot_2_left_wheel_joint: type continuous, parent robot_2_base_footprint, child robot_2_left_wheel, origin xyz=0 0.175 0 rpy=1.5707963267948966 0 0, axis 0 0 1
- added joint robot_2_right_wheel_joint: type continuous, parent robot_2_base_footprint, child robot_2_right_wheel, origin xyz=0 -0.175 0 rpy=1.5707963267948966 0 0, axis 0 0 1
